File: _autosave-ESP32-Based Sensor PCB.kicad_sch (KiCad schematic)
At the start: 51 parts, among them J1 USB_B_Micro, J2 rs485, J3 I2C, J4 UART_1, J5 ANALOG_IN, J6 9v OUT, J7 5v OUT, J8 3.3v OUT, Q1 MMBT3904LT1G, Q2 MMBT3906LT1G, Q3 MMBT3904LT1G, Q4 MMBT3904LT1G, Q5 MMBT3904LT1G, U1 ESP32-WROOM-32, U2 AMS1117-3.3, U3 CH340C, U4 USBLC6-2SC6, U5 TCA9548APWR, U6 MAX3485

Commit message: Fixed resistor size.
Parts:
- R7: footprint Resistor_SMD:R_0805_2012Metric -> Resistor_SMD:R_1206_3216Metric
Changed lines of the file:
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@@
 			)
 		)
-		(property "Footprint" "Resistor_SMD:R_0805_2012Metric"
+		(property "Footprint" "Resistor_SMD:R_1206_3216Metric"
 			(at 259.842 133.35 90)
 			(effects
